Commit message: ur3e simulation passed

File: cartesian_controller_simulation/urdf/ur3e/robot.urdf.xacro (robot description, xacro)
@@ -18,47 +18,24 @@
       visual_parameters_file="$(find ur_description)/config/ur3e/visual_parameters.yaml"
       use_fake_hardware="true"
-      sim_gazebo="true">
+      sim_gazebo="false">
     <origin xyz="0 0.0 0.0" rpy="0 0 0" />
   </xacro:ur_robot>
+  <xacro:include filename="$(find cartesian_controller_simulation)/urdf/joint.urdf.xacro"/>
   <ros2_control name="cartesian_controller_simulation" type="system">
+    <xacro:joint_interface name="shoulder_pan_joint" p="1000" d="0.5" />
+    <xacro:joint_interface name="shoulder_lift_joint" p="1000" d="0.5" />
+    <xacro:joint_interface name="elbow_joint" p="500" d="0.5" />
+    <xacro:joint_interface name="wrist_1_joint" p="100" d="0.5" />
+    <xacro:joint_interface name="wrist_2_joint" p="10" d="0.5" />
+    <xacro:joint_interface name="wrist_3_joint" p="10" d="0.5" />
     <hardware>
-        <plugin>cartesian_controller_simulation/Simulator</plugin>
-        <param name="mujoco_model">$(arg mujoco_model)</param>
+      <plugin>cartesian_controller_simulation/Simulator</plugin>
+      <param name="mujoco_model">$(arg mujoco_model)</param>
     </hardware>
-    <joint name="shoulder_pan_joint">
-      <command_interface name="position"/>
-      <state_interface name="position"/>
-      <state_interface name="velocity"/>
-    </joint>
-    <joint name="shoulder_lift_joint">
-      <command_interface name="position"/>
-      <state_interface name="position"/>
-      <state_interface name="velocity"/>
-    </joint>
-    <joint name="elbow_joint">
-      <command_interface name="position"/>
-      <state_interface name="position"/>
-      <state_interface name="velocity"/>
-    </joint>
-    <joint name="wrist_1_joint">
-      <command_interface name="position"/>
-      <state_interface name="position"/>
-      <state_interface name="velocity"/>
-    </joint>
-    <joint name="wrist_2_joint">
-      <command_interface name="position"/>
-      <state_interface name="position"/>
-      <state_interface name="velocity"/>
-    </joint>
-    <joint name="wrist_3_joint">
-      <command_interface name="position"/>
-      <state_interface name="position"/>
-      <state_interface name="velocity"/>
-    </joint>
   </ros2_control>
-  <gazebo>
+  <!-- <gazebo>
     <plugin filename="libgazebo_ros2_control.so" name="gazebo_ros2_control">
       <parameters>$(find ur_description)/config/initial_positions.yaml</parameters>
     </plugin>
-  </gazebo>
+  </gazebo> -->
 </robot>

Commit message: ur3e sim init pass

File: cartesian_controller_simulation/urdf/ur3e/robot.urdf.xacro (robot description, xacro)
@@ -3,5 +3,23 @@
   xmlns:xacro="http://ros.org/wiki/xacro">
   <xacro:include filename="$(find ur_description)/urdf/ur_macro.xacro" />
+  <!-- ur_type -->
+  <xacro:arg name="ur_type" default="ur3e"/>
+  <!-- ros2_control related parameters -->
   <xacro:arg name="robot_ip" default="192.168.1.101" />
+  <!-- parameters -->
+  <xacro:arg name="tf_prefix" default=""/>
+  <xacro:arg name="transmission_hw_interface" default=""/>
+  <xacro:arg name="safety_limits" default="false"/>
+  <xacro:arg name="safety_pos_margin" default="0.15"/>
+  <xacro:arg name="safety_k_position" default="20"/>
+  <!-- Simulation parameters -->
+  <xacro:arg name="use_fake_hardware" default="true" />
+  <xacro:arg name="fake_sensor_commands" default="false" />
+  <xacro:arg name="sim_gazebo" default="false" />
+  <xacro:arg name="sim_ignition" default="false" />
+  <xacro:arg name="simulation_controllers" default="" />
+  <!-- initial position for simulations (Fake Hardware, Gazebo, Ignition) -->
+  <xacro:arg name="initial_positions_file" default="$(find cartesian_controller_simulation)/config/initial_positions.yaml"/>
+  <xacro:property name="initial_positions_file" default="$(arg initial_positions_file)"/>
   <link name="world" />
   <joint name="world_joint" type="fixed">
@@ -10,13 +28,20 @@
     <child link="base_link" />
   </joint>
-  <xacro:ur_robot name="ur3e"
-      tf_prefix="" parent="world"
+  <xacro:ur_robot name="$(arg ur_type)"
       robot_ip="$(arg robot_ip)"
-      joint_limits_parameters_file="$(find ur_description)/config/ur3e/joint_limits.yaml"
-      kinematics_parameters_file="$(find ur_description)/config/ur3e/default_kinematics.yaml"
-      physical_parameters_file="$(find ur_description)/config/ur3e/physical_parameters.yaml"
-      visual_parameters_file="$(find ur_description)/config/ur3e/visual_parameters.yaml"
-      use_fake_hardware="true"
-      sim_gazebo="false">
+      tf_prefix="$(arg tf_prefix)" parent="world"
+      transmission_hw_interface="$(arg transmission_hw_interface)"
+      safety_limits="$(arg safety_limits)"
+      safety_pos_margin="$(arg safety_pos_margin)"
+      safety_k_position="$(arg safety_k_position)"
+      joint_limits_parameters_file="$(find ur_description)/config/$(arg ur_type)/joint_limits.yaml"
+      kinematics_parameters_file="$(find ur_description)/config/$(arg ur_type)/default_kinematics.yaml"
+      physical_parameters_file="$(find ur_description)/config/$(arg ur_type)/physical_parameters.yaml"
+      visual_parameters_file="$(find ur_description)/config/$(arg ur_type)/visual_parameters.yaml"
+      use_fake_hardware="$(arg use_fake_hardware)"
+      fake_sensor_commands="$(arg fake_sensor_commands)"
+      sim_gazebo="$(arg sim_gazebo)"
+      sim_ignition="$(arg sim_ignition)"
+      initial_positions="${xacro.load_yaml(initial_positions_file)}">
     <origin xyz="0 0.0 0.0" rpy="0 0 0" />
   </xacro:ur_robot>
@@ -39,3 +64,24 @@
     </plugin>
   </gazebo> -->
+  <xacro:if value="$(arg sim_gazebo)">
+    <!-- Gazebo plugins -->
+    <gazebo reference="world">
+    </gazebo>
+    <gazebo>
+      <plugin filename="libgazebo_ros2_control.so" name="gazebo_ros2_control">
+        <parameters>$(arg simulation_controllers)</parameters>
+      </plugin>
+    </gazebo>
+  </xacro:if>
+  <xacro:if value="$(arg sim_ignition)">
+    <!-- Gazebo plugins -->
+    <gazebo reference="world">
+    </gazebo>
+    <gazebo>
+      <plugin filename="libign_ros2_control-system.so" name="ign_ros2_control::IgnitionROS2ControlPlugin">
+        <parameters>$(arg simulation_controllers)</parameters>
+        <controller_manager_node_name>$(arg tf_prefix)controller_manager</controller_manager_node_name>
+      </plugin>
+    </gazebo>
+  </xacro:if>
 </robot>
